File: kicad_electronic_circuits/power_distribution_circuit/power_distribution_circuit.kicad_pcb (KiCad board)
At the start: 2 copper layers, 8 parts, among them J2 Conn_01x04, J3 Conn_01x02, J4 Conn_01x02, J5 Conn_01x04, J6 Conn_01x04, J7 Conn_01x02, J8 Conn_01x02, J9 Conn_01x04

Commit message: qu
Parts:
- added REF**: MountingHole_3.2mm_M3, MountingHole:MountingHole_3.2mm_M3, F.Cu at (105.4, 67.3)
- added REF**: MountingHole_3.2mm_M3, MountingHole:MountingHole_3.2mm_M3, F.Cu at (105.4, 110.5)
- added REF**: MountingHole_3.2mm_M3, MountingHole:MountingHole_3.2mm_M3, F.Cu at (174.0, 67.3)
- added REF**: MountingHole_3.2mm_M3, MountingHole:MountingHole_3.2mm_M3, F.Cu at (174.0, 110.5)
- moved J4 50.6 mm to (153.7, 74.0)
- moved J8 32.0 mm to (165.1, 104.1)
- moved J9 24.4 mm to (154.9, 86.4)
- moved J2 18.4 mm to (108.3, 90.2)
- moved J7 16.3 mm to (114.3, 104.1)
- moved J3 15.2 mm to (113.1, 74.0)
- moved J6 4.99 mm to (130.8, 86.4)
- moved J5 1.27 mm to (120.7, 86.4)
Other:
- board outline added: 76.2 x 50.8 mm

Commit message: more mods to circuit
Parts:
- added J1: Conn_01x02, TerminalBlock_Altech:Altech_AK100_1x02_P5.00mm, F.Cu at (117.3, 74.1)
- J2: footprint Connector_PinHeader_2.54mm:PinHeader_1x04_P2.54mm_Vertical_SMD_Pin1Right -> Connector_PinHeader_2.54mm:PinHeader_1x04_P2.54mm_Vertical
- moved J3 27.9 mm to (141.0, 74.0)
- moved J2 14.1 mm to (121.9, 86.4)
- moved J5 11.4 mm to (132.1, 86.4)
- moved J6 11.4 mm to (142.2, 86.4)
- moved REF** 1.80 mm to (106.7, 68.6)
- moved REF** 1.80 mm to (106.7, 109.2)
- moved REF** 1.80 mm to (172.7, 68.6)
- moved REF** 1.80 mm to (172.7, 109.2)
Routing:
- net +3.3V: track 0.00 -> 73.0 mm
- net /7.4V: track 0.00 -> 53.1 mm
- net /SDA: track 0.00 -> 20.3 mm
- net /SCL: track 0.00 -> 20.3 mm
- added copper zone on B.Cu, net GND

Commit message: modified power distribution circuit
Routing:
- net /7.4V: track 53.1 -> 53.8 mm
Changed lines of the file:
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@@
 		(capping no)
 		(filling no)
+		(zone_defaults)
 		(pcbplotparams
 			(layerselection 0x00000000_00000000_55555555_5755f5ff)
@@
 			(at 0 -4.15 0)
 			(layer "F.SilkS")
+			(hide yes)
 			(effects
 				(font
@@
 			(at 0 -4.15 0)
 			(layer "F.SilkS")
+			(hide yes)
 			(effects
 				(font
@@
 			(at 0 -4.15 0)
 			(layer "F.SilkS")
+			(hide yes)
 			(effects
 				(font
@@
 			(at 0 -4.15 0)
 			(layer "F.SilkS")
+			(hide yes)
 			(effects
 				(font
@@
 		(end 170.114269 84.732683)
 		(stroke
-			(width 0)
+			(width 0.1)
 			(type solid)
 		)
@@
 		(end 172.114269 84.89935)
 		(stroke
-			(width 0)
+			(width 0.1)
 			(type solid)
 		)
@@
 	)
 	(segment
-		(start 153.71 85.13)
-		(end 154.94 86.36)
-		(width 0.2)
+		(start 141.01 74.0275)
+		(end 143.9175 71.12)
+		(width 2)
 		(layer "F.Cu")
 		(net "/7.4V")
 	)
 	(segment
-		(start 117.325 74.105)
-		(end 119.125 72.305)
-		(width 0.2)
+		(start 153.71 74.0275)
+		(end 153.71 85.13)
+		(width 2)
 		(layer "F.Cu")
 		(net "/7.4V")
 	)
 	(segment
-		(start 153.71 74.0275)
-		(end 153.71 85.13)
-		(width 0.2)
+		(start 150.8025 71.12)
+		(end 153.71 74.0275)
+		(width 2)
 		(layer "F.Cu")
 		(net "/7.4V")
 	)
 	(segment
-		(start 141.01 74.0275)
-		(end 143.9175 71.12)
-		(width 0.2)
+		(start 143.9175 71.12)
+		(end 150.8025 71.12)
+		(width 2)
 		(layer "F.Cu")
 		(net "/7.4V")
 	)
 	(segment
-		(start 139.2875 72.305)
+		(start 138.3875 71.405)
 		(end 141.01 74.0275)
-		(width 0.2)
+		(width 2)
 		(layer "F.Cu")
 		(net "/7.4V")
 	)
 	(segment
-		(start 150.8025 71.12)
-		(end 153.71 74.0275)
-		(width 0.2)
+		(start 117.325 74.105)
+		(end 120.025 71.405)
+		(width 2)
 		(layer "F.Cu")
 		(net "/7.4V")
 	)
 	(segment
-		(start 119.125 72.305)
-		(end 139.2875 72.305)
-		(width 0.2)
+		(start 153.71 85.13)
+		(end 154.94 86.36)
+		(width 2)
 		(layer "F.Cu")
 		(net "/7.4V")
 	)
 	(segment
-		(start 143.9175 71.12)
-		(end 150.8025 71.12)
-		(width 0.2)
+		(start 120.025 71.405)
+		(end 138.3875 71.405)
+		(width 2)
 		(layer "F.Cu")
 		(net "/7.4V")
 	)
 	(segment
-		(start 149.86 86.36)
-		(end 154.94 91.44)
-		(width 0.2)
+		(start 121.92 86.36)
+		(end 114.3 93.98)
+		(width 0.5)
 		(layer "F.Cu")
 		(net "+3.3V")
 	)
 	(segment
-		(start 121.92 86.36)
-		(end 114.3 93.98)
-		(width 0.2)
+		(start 154.94 91.44)
+		(end 165.1 101.6)
+		(width 0.5)
 		(layer "F.Cu")
 		(net "+3.3V")
 	)
 	(segment
-		(start 132.08 86.36)
-		(end 142.24 86.36)
-		(width 0.2)
+		(start 165.1 101.6)
+		(end 165.1 104.14)
+		(width 0.5)
 		(layer "F.Cu")
 		(net "+3.3V")
 	)
 	(segment
-		(start 114.3 93.98)
-		(end 114.3 104.14)
-		(width 0.2)
+		(start 149.86 86.36)
+		(end 154.94 91.44)
+		(width 0.5)
 		(layer "F.Cu")
 		(net "+3.3V")
 	)
 	(segment
-		(start 165.1 101.6)
-		(end 165.1 104.14)
-		(width 0.2)
+		(start 142.24 86.36)
+		(end 149.86 86.36)
+		(width 0.5)
 		(layer "F.Cu")
 		(net "+3.3V")
 	)
 	(segment
-		(start 121.92 86.36)
-		(end 132.08 86.36)
-		(width 0.2)
+		(start 114.3 93.98)
+		(end 114.3 104.14)
+		(width 0.5)
 		(layer "F.Cu")
 		(net "+3.3V")
 	)
 	(segment
-		(start 142.24 86.36)
-		(end 149.86 86.36)
-		(width 0.2)
+		(start 121.92 86.36)
+		(end 132.08 86.36)
+		(width 0.5)
 		(layer "F.Cu")
 		(net "+3.3V")
 	)
 	(segment
-		(start 154.94 91.44)
-		(end 165.1 101.6)
-		(width 0.2)
+		(start 132.08 86.36)
+		(end 142.24 86.36)
+		(width 0.5)
 		(layer "F.Cu")
 		(net "+3.3V")
 	)
 	(segment
-		(start 121.92 88.9)
-		(end 132.08 88.9)
-		(width 0.2)
+		(start 132.08 88.9)
+		(end 142.24 88.9)
+		(width 0.25)
 		(layer "F.Cu")
 		(net "/SDA")
 	)
 	(segment
-		(start 132.08 88.9)
-		(end 142.24 88.9)
-		(width 0.2)
+		(start 121.92 88.9)
+		(end 132.08 88.9)
+		(width 0.25)
 		(layer "F.Cu")
 		(net "/SDA")
@@
 		(start 132.08 91.44)
 		(end 142.24 91.44)
-		(width 0.2)
+		(width 0.25)
 		(layer "F.Cu")
 		(net "/SCL")
@@
 		(start 121.92 91.44)
 		(end 132.08 91.44)
-		(width 0.2)
+		(width 0.25)
 		(layer "F.Cu")
 		(net "/SCL")
