File: kicad_electronic_circuits/power_distribution_circuit/power_distribution_circuit.kicad_sch (KiCad schematic)
At the start: 9 parts, among them J1 Conn_01x02, J2 Conn_01x04, J3 Conn_01x02, J4 Conn_01x02, J5 Conn_01x04, J6 Conn_01x04, J7 Conn_01x02, J8 Conn_01x02, J9 Conn_01x04

Commit message: more mods to circuit
Parts:
- J1: footprint (none) -> TerminalBlock_Altech:Altech_AK100_1x02_P5.00mm
- J2: footprint Connector_PinHeader_2.54mm:PinHeader_1x04_P2.54mm_Vertical_SMD_Pin1Right -> Connector_PinHeader_2.54mm:PinHeader_1x04_P2.54mm_Vertical
Changed lines of the file:
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@@
 			)
 		)
-		(property "Footprint" "Connector_PinHeader_2.54mm:PinHeader_1x04_P2.54mm_Vertical_SMD_Pin1Right"
+		(property "Footprint" "Connector_PinHeader_2.54mm:PinHeader_1x04_P2.54mm_Vertical"
 			(at 97.79 143.51 0)
 			(hide yes)
@@
 			)
 		)
-		(property "Footprint" ""
+		(property "Footprint" "TerminalBlock_Altech:Altech_AK100_1x02_P5.00mm"
 			(at 95.25 80.01 0)
 			(hide yes)

Commit message: qu
Parts:
- J1, J3, J4: MPN (none) -> 30.002; Manufacturer (none) -> Altech
- J2, J5, J6, J9: MPN (none) -> TSW-104-14-T-S; Manufacturer (none) -> Samtec
- J7, J8: MPN (none) -> TSW-102-14-T-S; Manufacturer (none) -> Samtec
