File: kicad_electronic_circuits/homebot_overview/homebot_overview.kicad_sch (KiCad schematic)
At the start: 5 parts, among them J1 Raspberry_Pi_4, M1 Motor_Servo, U1 TB6612FNG, U2 BNO055, U3 PCA9635

Commit message: doc update
Parts:
- removed M1: Motor_Servo, symbol Motor:Motor_Servo
- removed U3: PCA9635, Package_SO:TSSOP-28_4.4x9.7mm_P0.65mm, symbol Driver_LED:PCA9635
Connections:
- net at U1.15 (PWMB): now also J1.33 (GPIO13/PWM1)
- net at U1.16 (BIN2): now also J1.18 (GPIO24/SDIO_DAT0)
- net at U1.17 (BIN1): now also J1.16 (GPIO23/SDIO_CMD)
- net at U1.19 (STBY): now also J1.22 (GPIO25/SDIO_DAT1)
- net at U1.21 (AIN1): now also J1.11 (GPIO17/SPI1_~{CE1})
- net at U1.22 (AIN2): now also J1.13 (GPIO27/SDIO_DAT3)
- net at U1.23 (PWMA): now also J1.32 (GPIO12/PWM0)
Other:
- moved on the sheet: J1, U1, U2

Commit message: made some progress on overview schematic
Parts:
- added M1, M2: (no value), symbol homebot_symbols:TT_Motor_Encoder
- added U3: (no value), symbol homebot_symbols:RPLidarC1
- added U4: PCA9685BS, Package_DFN_QFN:QFN-28-1EP_6x6mm_P0.65mm_EP4.25x4.25mm, symbol Driver_LED:PCA9685BS
- added U5: (no value), symbol homebot_symbols:RPLIDAR_USB_ADAPTER
Connections:
- net at J1.29 (GPCLK1/GPIO05): now also M1.5 (A)
- net at J1.31 (GPCLK2/GPIO06): now also M1.6 (B)
- net at J1.36 (GPIO16/SPI1_~{CE2}): now also M2.5 (A)
- net at J1.37 (GPIO26/SDIO_DAT2): now also M2.6 (B)
- new net: U3.1 (VCC_5V), U5.1 (VCC_5V)
- new net: U3.2 (TX), U5.2 (TX)
- new net: U3.3 (RX), U5.3 (RX)
- new net: U3.4 (GND), U5.4 (GND)
Other:
- moved on the sheet: U2

Commit message: some progress, finish connections to pcn in homebot overview(take snapshots)
Parts:
- added PCB1: (no value), symbol homebot_symbols:Power_Distribution_PCB
Connections:
- net at J1.1 (3V3), J1.17 (3V3): now also PCB1.J2 (GND)
Changed lines of the file:
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@@
+	(wire
+		(pts
+			(xy 217.17 38.1) (xy 217.17 153.67)
+		)
+		(stroke
+			(width 0)
+			(type default)
+		)
+	)
 	(wire
 		(pts
@@
 	(wire
 		(pts
+			(xy 217.17 153.67) (xy 147.32 153.67)
+		)
+		(stroke
+			(width 0)
+			(type default)
+		)
+	)
+	(wire
+		(pts
 			(xy 44.45 118.11) (xy 52.07 118.11)
 		)
@@
 	(wire
 		(pts
+			(xy 147.32 153.67) (xy 147.32 161.29)
+		)
+		(stroke
+			(width 0)
+			(type default)
+		)
+	)
+	(wire
+		(pts
 			(xy 88.9 71.12) (xy 93.98 71.12)
+		)
+		(stroke
+			(width 0)
+			(type default)
+		)
+	)
+	(wire
+		(pts
+			(xy 160.02 38.1) (xy 217.17 38.1)
 		)
 		(stroke
@@
 					(unit 1)
 				)
+			)
+		)
+	)
+	(symbol
+		(lib_id "homebot_symbols:Power_Distribution_PCB")
+		(at 149.86 167.64 270)
+		(unit 1)
+		(body_style 1)
+		(exclude_from_sim no)
+		(in_bom yes)
+		(on_board yes)
+		(in_pos_files yes)
+		(dnp no)
+		(fields_autoplaced yes)
+		(property "Reference" "PCB1"
+			(at 160.02 172.7199 90)
+			(show_name no)
+			(do_not_autoplace no)
+			(effects
+				(font
+					(size 1.27 1.27)
+				)
+				(justify left)
+			)
+		)
+		(property "Value" ""
+			(at 149.86 167.64 0)
+			(show_name no)
+			(do_not_autoplace no)
+			(effects
+				(font
+					(size 1.27 1.27)
+				)
+			)
+		)
+		(property "Footprint" ""
+			(at 149.86 167.64 0)
+			(hide yes)
+			(show_name no)
+			(do_not_autoplace no)
+			(effects
+				(font
+					(size 1.27 1.27)
+				)
+			)
+		)
+		(property "Datasheet" ""
+			(at 149.86 167.64 0)
+			(hide yes)
+			(show_name no)
+			(do_not_autoplace no)
+			(effects
+				(font
+					(size 1.27 1.27)
+				)
+			)
+		)
+		(property "Description" ""
+			(at 149.86 167.64 0)
+			(hide yes)
+			(show_name no)
+			(do_not_autoplace no)
+			(effects
+				(font
+					(size 1.27 1.27)
+				)
+			)
+		)
+		(pin "J2"
+		)
+		(pin "J1"
+		)
+		(pin "J2"
+		)
+		(pin "J1"
+		)
+		(pin "J2"
+		)
+		(pin "J2"
+		)
+		(pin "J3"
+		)
+		(pin "J3"
+		)
+		(pin "J5"
+		)
+		(pin "J5"
+		)
+		(pin "J7"
+		)
+		(pin "J7"
+		)
+		(pin "J5"
+		)
+		(pin "J8"
+		)
+		(pin "J8"
+		)
+		(pin "J9"
+		)
+		(pin "J9"
+		)
+		(pin "J9"
+		)
+		(pin "J5"
+		)
+		(instances
+			(project "homebot_overview"
+				(path "/58295f61-e891-4a82-bc0b-1c626966d0f9"
+					(reference "PCB1")
+					(unit 1)
+				)

Commit message: wrapped up electrical overview
Parts:
- removed U2: BNO055, Package_LGA:LGA-28_5.2x3.8mm_P0.5mm, symbol Sensor_Motion:BNO055
- added P1: (no value), symbol homebot_symbols:Buck_converter_7.4V_to_5V
- added U2: (no value), symbol homebot_symbols:BNO055_Module
Connections:
- net at U1.1 (AO1), U1.2 (AO1): now also M1.1 (MOTOR+)
- net at U1.11 (BO1), U1.12 (BO1): now also M2.1 (MOTOR+)
- net at U1.18 (GND): now also PCB1.J9 (GND)
- net at U1.20 (VCC): now also PCB1.J9 (GND)
- net at U1.24 (VM1): now also PCB1.J9 (GND)
- net at U1.5 (AO2), U1.6 (AO2): now also M1.2 (MOTOR-)
- net at U1.7 (BO2), U1.8 (BO2): now also M2.2 (MOTOR-)
- net at PCB1.J2 (GND): now also J1.5 (SCL_I2C1/GPIO03)
- net at PCB1.J3 (GND): now also P1.2 (GND)
- net at PCB1.J5 (GND): now also U2.4 (GND)
- net at PCB1.J7 (GND): now also M1.4 (GND)
- net at PCB1.J8 (GND): now also M2.4 (GND)
- net at J1.14 (GND), J1.20 (GND), J1.25 (GND)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: now also PCB1.J2 (GND)
- net at J1.3 (SDA_I2C1/GPIO02): now also PCB1.J2 (GND)
- net at M1.3 (VCC): now also PCB1.J7 (GND)
- net at M2.3 (VCC): now also PCB1.J8 (GND)
- new net: P1.1 (7.4V), PCB1.J3 (GND)
- new net: PCB1.J5 (GND), U2.1 (3.3V)
- new net: PCB1.J5 (GND), U2.2 (SDA)
- new net: PCB1.J5 (GND), U2.3 (SCL)
