Commit message: messing with urdf model some more

File: ros2_ws/src/my_robot_description/urdf/my_robot.urdf.xacro (robot description, xacro)
@@ -53,4 +53,7 @@
         </geometry>
         <origin rpy="1.5708 0 0"/>
+        <material name="black">
+            <color rgba="0 0 0 1"/>
+        </material>
     </visual>
     <collision>
@@ -86,4 +89,7 @@
             <sphere radius="0.015"/>
         </geometry>
+        <material name="gray">
+            <color rgba=".35 .35 .35 1"/>
+        </material>
     </visual>
     <collision>
@@ -107,4 +113,7 @@
             <box size="0.01 0.01 0.005"/>
         </geometry>
+        <material name="blue">
+            <color rgba="0 0 .5 1"/>
+        </material>
     </visual>
 </link>
@@ -123,4 +132,7 @@
             <box size="0.015 0.015 0.015"/>
         </geometry>
+        <material name="red">
+            <color rgba="1 0 0 1"/>
+        </material>
     </visual>
 </link>
@@ -140,4 +152,7 @@
                   scale="0.001 0.001 0.001"/>
         </geometry>
+        <material name="gray">
+            <color rgba=".35 .35 .35 1"/>
+        </material>
     </visual>
     <collision>
@@ -148,4 +163,5 @@
     </collision>
 </link>
+<!-- Servo enclosure is fixed to robot -->
 <joint name="lidar_base_joint" type="fixed">
     <parent link="base_link"/>
@@ -155,7 +171,7 @@
 </joint>
 <!-- ========================= -->
-<!-- Rotating LiDAR cover      -->
-<!-- ========================= -->
-<link name="lidar_cover_link">
+<!-- Stationary Base Cover     -->
+<!-- ========================= -->
+<link name="base_cover_link">
     <visual>
         <geometry>
@@ -163,10 +179,34 @@
                   scale="0.001 0.001 0.001"/>
         </geometry>
-    </visual>
-</link>
+        <material name="white">
+            <color rgba="1 1 1 1"/>
+        </material>
+    </visual>
+</link>
+<joint name="base_cover_joint" type="fixed">
+    <parent link="base_link"/>
+    <child link="base_cover_link"/>
+    <origin xyz="0 0 0.055"
+            rpy="0 0 0"/>
+</joint>
+<!-- ========================= -->
+<!-- Rotating LiDAR            -->
+<!-- ========================= -->
+<link name="lidar_link">
+    <visual>
+        <geometry>
+            <cylinder radius="0.03"
+                      length="0.02"/>
+        </geometry>
+        <material name="black">
+            <color rgba="0 1 0 1"/>
+        </material>
+    </visual>
+</link>
+<!-- Servo shaft rotates lidar -->
 <joint name="lidar_rotation_joint" type="revolute">
     <parent link="lidar_base_link"/>
-    <child link="lidar_cover_link"/>
-    <origin xyz="0 0 0"
+    <child link="lidar_link"/>
+    <origin xyz="0 0 0.045"
             rpy="0 0 0"/>
     <axis xyz="0 0 1"/>
@@ -177,20 +217,3 @@
         velocity="5"/>
 </joint>
-<!-- ========================= -->
-<!-- LiDAR Sensor              -->
-<!-- ========================= -->
-<link name="lidar_link">
-    <visual>
-        <geometry>
-            <cylinder radius="0.03"
-                      length="0.02"/>
-        </geometry>
-    </visual>
-</link>
-<joint name="lidar_joint" type="fixed">
-    <parent link="lidar_cover_link"/>
-    <child link="lidar_link"/>
-    <origin xyz="0 0 0.025"
-            rpy="0 0 0"/>
-</joint>
 </robot>

Commit message: fixing up robot position of links and joints in urdf

File: ros2_ws/src/my_robot_description/urdf/my_robot.urdf.xacro (robot description, xacro)
@@ -2,7 +2,5 @@
 <robot xmlns:xacro="http://www.ros.org/wiki/xacro"
        name="my_robot">
-<!-- ========================= -->
 <!-- Properties                -->
-<!-- ========================= -->
 <xacro:property name="base_length" value="0.1500"/>
 <xacro:property name="base_width"  value="0.1250"/>
@@ -10,9 +8,8 @@
 <xacro:property name="wheel_radius" value="0.0205"/>
 <xacro:property name="wheel_width"  value="0.017"/>
-<xacro:property name="wheel_x" value="-0.06985"/>
-<xacro:property name="wheel_y" value="0.072"/>
-<!-- ========================= -->
+<xacro:property name="wheel_x" value="0.0225"/>
+<xacro:property name="left_wheel_y" value="0.1335"/>
+<xacro:property name="right_wheel_y" value="-0.0085"/>
 <!-- Base                      -->
-<!-- ========================= -->
 <link name="base_link">
     <visual>
@@ -42,7 +39,5 @@
     </inertial>
 </link>
-<!-- ========================= -->
 <!-- Wheels                    -->
-<!-- ========================= -->
 <xacro:macro name="wheel" params="name x y">
 <link name="${name}">
@@ -68,5 +63,5 @@
     <parent link="base_link"/>
     <child link="${name}"/>
-    <origin xyz="${x} ${y} ${wheel_radius}"
+    <origin xyz="${x} ${y} -0.0105"
             rpy="0 0 0"/>
     <axis xyz="0 1 0"/>
@@ -76,12 +71,10 @@
     name="left_wheel"
     x="${wheel_x}"
-    y="${wheel_y}"/>
+    y="${left_wheel_y}"/>
 <xacro:wheel
     name="right_wheel"
     x="${wheel_x}"
-    y="-${wheel_y}"/>
-<!-- ========================= -->
+    y="${right_wheel_y}"/>
 <!-- Front Caster               -->
-<!-- ========================= -->
 <link name="caster_link">
     <visual>
@@ -102,10 +95,8 @@
     <parent link="base_link"/>
     <child link="caster_link"/>
-    <origin xyz="0.0762 0 -0.005"
-            rpy="0 0 0"/>
-</joint>
-<!-- ========================= -->
+    <origin xyz="0.140 0.0625 -0.01"
+            rpy="0 0 0"/>
+</joint>
 <!-- MPU6050 IMU               -->
-<!-- ========================= -->
 <link name="imu_link">
     <visual>
@@ -113,6 +104,6 @@
             <box size="0.01 0.01 0.005"/>
         </geometry>
-        <material name="blue">
-            <color rgba="0 0 .5 1"/>
+        <material name="light blue">
+            <color rgba="0 0 .25 1"/>
         </material>
     </visual>
@@ -121,10 +112,8 @@
     <parent link="base_link"/>
     <child link="imu_link"/>
-    <origin xyz="-0.06985 0.072 0.0459"
-            rpy="0 0 0"/>
-</joint>
-<!-- ========================= -->
+    <origin xyz="0.02 0 0.0459"
+            rpy="0 0 0"/>
+</joint>
 <!-- Camera                    -->
-<!-- ========================= -->
 <link name="camera_link">
     <visual>
@@ -140,10 +129,8 @@
     <parent link="base_link"/>
     <child link="camera_link"/>
-    <origin xyz="0.0762 0.04445 0.075"
-            rpy="0 0 0"/>
-</joint>
-<!-- ========================= -->
+    <origin xyz="0.142 .02 0.035"
+            rpy="0 0 0"/>
+</joint>
 <!-- LiDAR Servo Housing       -->
-<!-- ========================= -->
 <link name="lidar_base_link">
     <visual>
@@ -167,10 +154,8 @@
     <parent link="base_link"/>
     <child link="lidar_base_link"/>
-    <origin xyz="0 0 0.075"
-            rpy="0 0 0"/>
-</joint>
-<!-- ========================= -->
+    <origin xyz=".05 .143 -0.0625"
+            rpy="1.5708 0 0"/>
+</joint>
 <!-- Stationary Base Cover     -->
-<!-- ========================= -->
 <link name="base_cover_link">
     <visual>
@@ -187,10 +172,8 @@
     <parent link="base_link"/>
     <child link="base_cover_link"/>
-    <origin xyz="0 0 0.055"
-            rpy="0 0 0"/>
-</joint>
-<!-- ========================= -->
+    <origin xyz="0 0 0.050"
+            rpy="0 0 0"/>
+</joint>
 <!-- Rotating LiDAR            -->
-<!-- ========================= -->
 <link name="lidar_link">
     <visual>
@@ -208,6 +191,6 @@
     <parent link="lidar_base_link"/>
     <child link="lidar_link"/>
-    <origin xyz="0 0 0.045"
-            rpy="0 0 0"/>
+    <origin xyz=".03 .125 .0855"
+            rpy="-1.5708 0 0"/>
     <axis xyz="0 0 1"/>
     <limit

Commit message: fixed homebot in rviz thru urdf

File: ros2_ws/src/my_robot_description/urdf/my_robot.urdf.xacro (robot description, xacro)
@@ -121,6 +121,6 @@
             <box size="0.015 0.015 0.015"/>
         </geometry>
-        <material name="red">
-            <color rgba="1 0 0 1"/>
+        <material name="green">
+            <color rgba="0 1 0 1"/>
         </material>
     </visual>
@@ -176,5 +176,5 @@
 </joint>
 <!-- Rotating LiDAR            -->
-<link name="lidar_link">
+<link name="servo_link">
     <visual>
         <geometry>
@@ -188,15 +188,32 @@
 </link>
 <!-- Servo shaft rotates lidar -->
-<joint name="lidar_rotation_joint" type="revolute">
+<joint name="servo_rotation_joint" type="revolute">
     <parent link="lidar_base_link"/>
-    <child link="lidar_link"/>
-    <origin xyz=".03 .125 .0855"
+    <child link="servo_link"/>
+    <origin xyz=".04 .125 .0875"
             rpy="-1.5708 0 0"/>
     <axis xyz="0 0 1"/>
     <limit
-        lower="-3.14159"
-        upper="3.14159"
+        lower="-1.5708"
+        upper="1.5708"
         effort="2"
         velocity="5"/>
 </joint>
+<link name="lidar_link">
+    <visual>
+        <geometry>
+            <box size="0.08 0.01 0.01"/>
+        </geometry>
+        <origin xyz="0.04 0 0"/>
+        <material name="red">
+            <color rgba="1 0 0 1"/>
+        </material>
+    </visual>
+</link>
+<joint name="lidar_joint" type="fixed">
+    <parent link="servo_link"/>
+    <child link="lidar_link"/>
+    <origin xyz="0 0 0.02"
+            rpy="0 0 0"/>
+</joint>
 </robot>

Commit message: adding top, still adjusting

File: ros2_ws/src/my_robot_description/urdf/my_robot.urdf.xacro (robot description, xacro)
@@ -179,5 +179,5 @@
     <visual>
         <geometry>
-            <cylinder radius="0.03"
+            <cylinder radius="0.02"
                       length="0.02"/>
         </geometry>
@@ -195,24 +195,41 @@
     <axis xyz="0 0 1"/>
     <limit
-        lower="-1.5708"
-        upper="1.5708"
+        lower="-3.14"
+        upper="3.14"
         effort="2"
         velocity="5"/>
 </joint>
+<link name="top_link">
+    <visual>
+        <geometry>
+            <mesh filename="package://my_robot_description/meshes/top.stl"
+                  scale="0.001 0.001 0.001"/>
+        </geometry>
+        <material name="gray">
+            <color rgba=".35 .35 .35 1"/>
+        </material>
+    </visual>
+</link>
+<joint name="top_joint" type="fixed">
+    <parent link="servo_link"/>
+    <child link="top_link"/>
+    <origin xyz="-.04 .09 -.125"
+            rpy="1.5708 0 0"/>
+</joint>
 <link name="lidar_link">
     <visual>
         <geometry>
-            <box size="0.08 0.01 0.01"/>
-        </geometry>
-        <origin xyz="0.04 0 0"/>
-        <material name="red">
-            <color rgba="1 0 0 1"/>
+            <box size="0.02125 0.035 0.012"/>
+        </geometry>
+        <origin xyz="0 0 0"/>
+        <material name="black">
+            <color rgba="0 0 0 1"/>
         </material>
     </visual>
 </link>
 <joint name="lidar_joint" type="fixed">
-    <parent link="servo_link"/>
+    <parent link="top_link"/>
     <child link="lidar_link"/>
-    <origin xyz="0 0 0.02"
+    <origin xyz="0 .15 .11"
             rpy="0 0 0"/>
 </joint>

Commit message: fit top, updated tfframe and sample gif

File: ros2_ws/src/my_robot_description/urdf/my_robot.urdf.xacro (robot description, xacro)
@@ -83,5 +83,5 @@
         </geometry>
         <material name="gray">
-            <color rgba=".35 .35 .35 1"/>
+            <color rgba=".5 .5 .5 1"/>
         </material>
     </visual>
@@ -122,5 +122,5 @@
         </geometry>
         <material name="green">
-            <color rgba="0 1 0 1"/>
+            <color rgba=".2 .2 .2 1"/>
         </material>
     </visual>
@@ -140,5 +140,5 @@
         </geometry>
         <material name="gray">
-            <color rgba=".35 .35 .35 1"/>
+            <color rgba=".5 .5 .5 1"/>
         </material>
     </visual>
@@ -165,5 +165,5 @@
         </geometry>
         <material name="white">
-            <color rgba="1 1 1 1"/>
+            <color rgba="1 1 1 .25"/>
         </material>
     </visual>
@@ -195,6 +195,6 @@
     <axis xyz="0 0 1"/>
     <limit
-        lower="-3.14"
-        upper="3.14"
+        lower="-2.6"
+        upper="-.4"
         effort="2"
         velocity="5"/>
@@ -207,5 +207,5 @@
         </geometry>
         <material name="gray">
-            <color rgba=".35 .35 .35 1"/>
+            <color rgba=".5 .5 .5 1"/>
         </material>
     </visual>
@@ -214,5 +214,5 @@
     <parent link="servo_link"/>
     <child link="top_link"/>
-    <origin xyz="-.04 .09 -.125"
+    <origin xyz="-.0375 .085 -.125"
             rpy="1.5708 0 0"/>
 </joint>
@@ -231,5 +231,5 @@
     <parent link="top_link"/>
     <child link="lidar_link"/>
-    <origin xyz="0 .15 .11"
+    <origin xyz=".04 .17 .09"
             rpy="0 0 0"/>
 </joint>

Commit message: updated lidar position on base, prepping for laserscan

File: ros2_ws/src/my_robot_description/urdf/my_robot.urdf.xacro (robot description, xacro)
@@ -231,6 +231,6 @@
     <parent link="top_link"/>
     <child link="lidar_link"/>
-    <origin xyz=".04 .17 .09"
-            rpy="0 0 0"/>
+    <origin xyz=".04 .2 .09"
+            rpy="0 0 .785"/>
 </joint>
 </robot>

Commit message: testing lasercan and top_link orientration complete

File: ros2_ws/src/my_robot_description/urdf/my_robot.urdf.xacro (robot description, xacro)
@@ -60,5 +60,6 @@
     </collision>
 </link>
-<joint name="${name}_joint" type="continuous">
+<!-- change type to continuous when moving -->
+<joint name="${name}_joint" type="fixed">
     <parent link="base_link"/>
     <child link="${name}"/>
@@ -92,4 +93,5 @@
     </collision>
 </link>
+<!-- change type to continuous when moving -->
 <joint name="caster_joint" type="fixed">
     <parent link="base_link"/>

Commit message: qc

File: ros2_ws/src/my_robot_description/urdf/my_robot.urdf.xacro (robot description, xacro)
@@ -2,5 +2,4 @@
 <robot xmlns:xacro="http://www.ros.org/wiki/xacro"
        name="my_robot">
-<!-- Properties                -->
 <xacro:property name="base_length" value="0.1500"/>
 <xacro:property name="base_width"  value="0.1250"/>
@@ -11,5 +10,4 @@
 <xacro:property name="left_wheel_y" value="0.1335"/>
 <xacro:property name="right_wheel_y" value="-0.0085"/>
-<!-- Base                      -->
 <link name="base_link">
     <visual>
@@ -60,6 +58,5 @@
     </collision>
 </link>
-<!-- change type to continuous when moving -->
-<joint name="${name}_joint" type="fixed">
+<joint name="${name}_joint" type="continuous">
     <parent link="base_link"/>
     <child link="${name}"/>
@@ -77,5 +74,4 @@
     x="${wheel_x}"
     y="${right_wheel_y}"/>
-<!-- Front Caster               -->
 <link name="caster_link">
     <visual>
@@ -93,5 +89,4 @@
     </collision>
 </link>
-<!-- change type to continuous when moving -->
 <joint name="caster_joint" type="fixed">
     <parent link="base_link"/>
@@ -100,5 +95,4 @@
             rpy="0 0 0"/>
 </joint>
-<!-- MPU6050 IMU               -->
 <link name="imu_link">
     <visual>
@@ -117,5 +111,4 @@
             rpy="0 0 0"/>
 </joint>
-<!-- Camera                    -->
 <link name="camera_link">
     <visual>
@@ -134,5 +127,4 @@
             rpy="0 0 0"/>
 </joint>
-<!-- LiDAR Servo Housing       -->
 <link name="lidar_base_link">
     <visual>
@@ -152,5 +144,4 @@
     </collision>
 </link>
-<!-- Servo enclosure is fixed to robot -->
 <joint name="lidar_base_joint" type="fixed">
     <parent link="base_link"/>
@@ -159,5 +150,4 @@
             rpy="1.5708 0 0"/>
 </joint>
-<!-- Stationary Base Cover     -->
 <link name="base_cover_link">
     <visual>
@@ -177,5 +167,4 @@
             rpy="0 0 0"/>
 </joint>
-<!-- Rotating LiDAR            -->
 <link name="servo_link">
     <visual>
@@ -189,5 +178,4 @@
     </visual>
 </link>
-<!-- Servo shaft rotates lidar -->
 <joint name="servo_rotation_joint" type="revolute">
     <parent link="lidar_base_link"/>

Commit message: added arm for homebot in urdf

File: ros2_ws/src/my_robot_description/urdf/my_robot.urdf.xacro (robot description, xacro)
@@ -224,3 +224,211 @@
             rpy="0 0 .785"/>
 </joint>
+<link name="shoulder_link">
+    <visual>
+        <geometry>
+            <mesh filename="package://my_robot_description/meshes/shoulder_small.stl"
+                  scale="0.001 0.001 0.001"/>
+        </geometry>
+        <material name="gray">
+            <color rgba="1 1 1 1"/>
+        </material>
+    </visual>
+    <collision>
+        <geometry>
+            <mesh filename="package://my_robot_description/meshes/shoulder_small.stl"
+                  scale="0.001 0.001 0.001"/>
+        </geometry>
+    </collision>
+</link>
+<joint name="shoulder_joint" type="fixed">
+    <parent link="top_link"/>
+    <child link="shoulder_link"/>
+    <origin xyz="0 0 0"
+            rpy="0 0 0"/>
+</joint>
+<link name="elbow_link">
+    <visual>
+        <geometry>
+            <mesh filename="package://my_robot_description/meshes/elbow_small.stl"
+                  scale="0.001 0.001 0.001"/>
+        </geometry>
+        <material name="gray">
+            <color rgba="1 1 1 1"/>
+        </material>
+    </visual>
+    <collision>
+        <geometry>
+            <mesh filename="package://my_robot_description/meshes/elbow_small.stl"
+                  scale="0.001 0.001 0.001"/>
+        </geometry>
+    </collision>
+</link>
+<joint name="elbow_joint" type="fixed">
+    <parent link="shoulder_link"/>
+    <child link="elbow_link"/>
+    <origin xyz="0 0 0"
+            rpy="0 0 0"/>
+</joint>
+<!-- when testing arm, make wheel joints and servo joint fixed -->
+<!-- <link name="base_gripper_link">
+    <visual>
+        <geometry>
+            <mesh filename="package://my_robot_description/meshes/base_gripper.stl"
+                  scale="0.001 0.001 0.001"/>
+        </geometry>
+        <material name="gray">
+            <color rgba="1 1 1 1"/>
+        </material>
+    </visual>
+    <collision>
+        <geometry>
+            <mesh filename="package://my_robot_description/meshes/base_gripper.stl"
+                  scale="0.001 0.001 0.001"/>
+        </geometry>
+    </collision>
+</link>
+<joint name="base_gripper_joint" type="fixed">
+    <parent link="elbow_link"/>
+    <child link="base_gripper_link"/>
+    <origin xyz="-.03 .155 .045"
+            rpy="0 0 0"/>
+</joint>
+<link name="gear1_link">
+    <visual>
+        <geometry>
+            <mesh filename="package://my_robot_description/meshes/gear1.stl"
+                  scale="0.001 0.001 0.001"/>
+        </geometry>
+        <material name="gray">
+            <color rgba="1 1 1 1"/>
+        </material>
+    </visual>
+    <collision>
+        <geometry>
+            <mesh filename="package://my_robot_description/meshes/gear1.stl"
+                  scale="0.001 0.001 0.001"/>
+        </geometry>
+    </collision>
+</link>
+<joint name="gear1_joint" type="fixed">
+    <parent link="base_gripper_link"/>
+    <child link="gear1_link"/>
+    <origin xyz="0 0 0"
+            rpy="0 0 0"/>
+</joint>
+<link name="gear2_link">
+    <visual>
+        <geometry>
+            <mesh filename="package://my_robot_description/meshes/gear2.stl"
+                  scale="0.001 0.001 0.001"/>
+        </geometry>
+        <material name="gray">
+            <color rgba="1 1 1 1"/>
+        </material>
+    </visual>
+    <collision>
+        <geometry>
+            <mesh filename="package://my_robot_description/meshes/gear2.stl"
+                  scale="0.001 0.001 0.001"/>
+        </geometry>
+    </collision>
+</link>
+<joint name="gear2_joint" type="fixed">
+    <parent link="base_gripper_link"/>
+    <child link="gear2_link"/>
+    <origin xyz="0 0 0"
+            rpy="0 0 0"/>
+</joint>
+<link name="bar1_link">
+    <visual>
+        <geometry>
+            <mesh filename="package://my_robot_description/meshes/bar1.stl"
+                  scale="0.001 0.001 0.001"/>
+        </geometry>
+        <material name="gray">
+            <color rgba="1 1 1 1"/>
+        </material>
+    </visual>
+    <collision>
+        <geometry>
+            <mesh filename="package://my_robot_description/meshes/bar1.stl"
+                  scale="0.001 0.001 0.001"/>
+        </geometry>
+    </collision>
+</link>
+<joint name="bar1_joint" type="fixed">
+    <parent link="base_gripper_link"/>
+    <child link="bar1_link"/>
+    <origin xyz="0 0 0"
+            rpy="0 0 0"/>
+</joint>
+<link name="bar2_link">
+    <visual>
+        <geometry>
+            <mesh filename="package://my_robot_description/meshes/bar2.stl"
+                  scale="0.001 0.001 0.001"/>
+        </geometry>
+        <material name="gray">
+            <color rgba="1 1 1 1"/>
+        </material>
+    </visual>
+    <collision>
+        <geometry>
+            <mesh filename="package://my_robot_description/meshes/bar2.stl"
+                  scale="0.001 0.001 0.001"/>
+        </geometry>
+    </collision>
+</link>
+<joint name="bar2_joint" type="fixed">
+    <parent link="base_gripper_link"/>
+    <child link="bar2_link"/>
+    <origin xyz="0 0 0"
+            rpy="0 0 0"/>
+</joint>
+<link name="gripper1_link">
+    <visual>
+        <geometry>
+            <mesh filename="package://my_robot_description/meshes/gripper1.stl"
+                  scale="0.001 0.001 0.001"/>
+        </geometry>
+        <material name="gray">
+            <color rgba="1 1 1 1"/>
+        </material>
+    </visual>
+    <collision>
+        <geometry>
+            <mesh filename="package://my_robot_description/meshes/gripper1.stl"
+                  scale="0.001 0.001 0.001"/>
+        </geometry>
+    </collision>
+</link>
+<joint name="gripper1_joint" type="fixed">
+    <parent link="base_gripper_link"/>
+    <child link="gripper1_link"/>
+    <origin xyz="0 0 0"
+            rpy="0 0 0"/>
+</joint>
+<link name="gripper2_link">
+    <visual>
+        <geometry>
+            <mesh filename="package://my_robot_description/meshes/gripper2.stl"
+                  scale="0.001 0.001 0.001"/>
+        </geometry>
+        <material name="gray">
+            <color rgba="1 1 1 1"/>
+        </material>
+    </visual>
+    <collision>
+        <geometry>
+            <mesh filename="package://my_robot_description/meshes/gripper2.stl"
+                  scale="0.001 0.001 0.001"/>
+        </geometry>
+    </collision>
+</link>
+<joint name="gripper2_joint" type="fixed">
+    <parent link="base_gripper_link"/>
+    <child link="gripper2_link"/>
+    <origin xyz="0 0 0"
+            rpy="0 0 0"/>
+</joint> -->
 </robot>
