Commit message: added marker to see wheels rotating, plus some more stuff on publishing joint state for wheels still gotta test

File: ros2_ws/src/my_robot_description/urdf/my_robot.urdf.xacro (robot description, xacro)
@@ -37,32 +37,42 @@
     </inertial>
 </link>
-<!-- Wheels                    -->
 <xacro:macro name="wheel" params="name x y">
-<link name="${name}">
-    <visual>
-        <geometry>
-            <cylinder radius="${wheel_radius}"
-                      length="${wheel_width}"/>
-        </geometry>
-        <origin rpy="1.5708 0 0"/>
-        <material name="black">
-            <color rgba="0 0 0 1"/>
-        </material>
-    </visual>
-    <collision>
-        <geometry>
-            <cylinder radius="${wheel_radius}"
-                      length="${wheel_width}"/>
-        </geometry>
-        <origin rpy="1.5708 0 0"/>
-    </collision>
-</link>
-<joint name="${name}_joint" type="continuous">
-    <parent link="base_link"/>
-    <child link="${name}"/>
-    <origin xyz="${x} ${y} -0.0105"
-            rpy="0 0 0"/>
-    <axis xyz="0 1 0"/>
-</joint>
+    <link name="${name}">
+        <visual>
+            <geometry>
+                <cylinder radius="${wheel_radius}"
+                          length="${wheel_width}"/>
+            </geometry>
+            <origin rpy="1.5708 0 0"/>
+            <material name="black">
+                <color rgba="0 0 0 1"/>
+            </material>
+        </visual>
+        <!-- Rotation marker -->
+        <visual>
+            <geometry>
+                <box size="0.006 0.006 0.025"/>
+            </geometry>
+            <origin xyz="${wheel_radius + 0.004} 0 0"
+                    rpy="0 0 0"/>
+            <material name="${name}_red_marker">
+                <color rgba="1 0 0 1"/>
+            </material>
+        </visual>
+        <collision>
+            <geometry>
+                <cylinder radius="${wheel_radius}"
+                          length="${wheel_width}"/>
+            </geometry>
+            <origin rpy="1.5708 0 0"/>
+        </collision>
+    </link>
+    <joint name="${name}_joint" type="continuous">
+        <parent link="base_link"/>
+        <child link="${name}"/>
+        <origin xyz="${x} ${y} -0.0105"
+                rpy="0 0 0"/>
+        <axis xyz="0 1 0"/>
+    </joint>
 </xacro:macro>
 <xacro:wheel
@@ -224,5 +234,6 @@
             rpy="0 0 .785"/>
 </joint>
-<link name="shoulder_link">
+<!-- when testing arm, make wheel joints and servo joint fixed -->
+<!-- <link name="shoulder_link">
     <visual>
         <geometry>
@@ -270,6 +281,5 @@
             rpy="0 0 0"/>
 </joint>
-<!-- when testing arm, make wheel joints and servo joint fixed -->
-<!-- <link name="base_gripper_link">
+<link name="base_gripper_link">
     <visual>
         <geometry>

Commit message: added rplidar to urdf

File: ros2_ws/src/my_robot_description/urdf/my_robot.urdf.xacro (robot description, xacro)
@@ -137,5 +137,39 @@
             rpy="0 0 0"/>
 </joint>
-<link name="lidar_base_link">
+<link name="base_cover_link">
+    <visual>
+        <geometry>
+            <mesh filename="package://my_robot_description/meshes/base_cover.stl"
+                  scale="0.001 0.001 0.001"/>
+        </geometry>
+        <material name="white">
+            <color rgba="1 1 1 .25"/>
+        </material>
+    </visual>
+</link>
+<joint name="base_cover_joint" type="fixed">
+    <parent link="base_link"/>
+    <child link="base_cover_link"/>
+    <origin xyz="0 0 0.050"
+            rpy="0 0 0"/>
+</joint>
+<link name="rplidar_link">
+    <visual>
+        <geometry>
+            <mesh filename="package://my_robot_description/meshes/rplidar.stl"
+                  scale="0.001 0.001 0.001"/>
+        </geometry>
+        <material name="black">
+            <color rgba="0 0 0 .75"/>
+        </material>
+    </visual>
+</link>
+<joint name="rplidar_joint" type="fixed">
+    <parent link="base_cover_link"/>
+    <child link="rplidar_link"/>
+    <origin xyz=".08 .07 .002"
+            rpy="0 0 0"/>
+</joint>
+<!-- <link name="lidar_base_link">
     <visual>
         <geometry>
@@ -159,21 +193,4 @@
     <origin xyz=".05 .143 -0.0625"
             rpy="1.5708 0 0"/>
-</joint>
-<link name="base_cover_link">
-    <visual>
-        <geometry>
-            <mesh filename="package://my_robot_description/meshes/base_cover.stl"
-                  scale="0.001 0.001 0.001"/>
-        </geometry>
-        <material name="white">
-            <color rgba="1 1 1 .25"/>
-        </material>
-    </visual>
-</link>
-<joint name="base_cover_joint" type="fixed">
-    <parent link="base_link"/>
-    <child link="base_cover_link"/>
-    <origin xyz="0 0 0.050"
-            rpy="0 0 0"/>
 </joint>
 <link name="servo_link">
@@ -234,6 +251,5 @@
             rpy="0 0 .785"/>
 </joint>
-<!-- when testing arm, make wheel joints and servo joint fixed -->
-<!-- <link name="shoulder_link">
+<link name="shoulder_link">
     <visual>
         <geometry>

Commit message: added laser frame to urdf

File: ros2_ws/src/my_robot_description/urdf/my_robot.urdf.xacro (robot description, xacro)
@@ -171,4 +171,11 @@
             rpy="0 0 0"/>
 </joint>
+<link name="laser"/>
+<joint name="laser_joint" type="fixed">
+    <parent link="rplidar_link"/>
+    <child link="laser"/>
+    <origin xyz="0 0 0"
+            rpy="0 0 0"/>
+</joint>
 <!-- <link name="lidar_base_link">
     <visual>
